File: files/eagle/sduino/sduino.brd (EAGLE design)
At the start: 100 x 80 mm, 13 parts, among them IC1 ATMEGA48/88/168-AU

Commit message: typo
Parts:
- removed JP2: (no value), fab:2X03SMD
- added JP1: (no value), pinhead:2X03
Connections:
- removed net N$16: IC1.8, U$2.3
- new net N$9: IC1.7, U$2.3
- net GND: now also JP1.6; no longer JP2.6
- net MISO: now also JP1.1; no longer JP2.1
- net MOSI: now also JP1.4; no longer JP2.4
- net N$1: now also IC1.8; no longer IC1.7
- net RST: now also JP1.5; no longer JP2.5
- net SCK: now also JP1.3; no longer JP2.3
- net VCC: now also JP1.2; no longer JP2.2
Routing:
- net N$9: track 0.00 -> 6.89 mm
- net N$1: track 0.00 -> 4.91 mm
- net S$1: track 0.00 -> 2.95 mm
- net MISO: track 29.7 -> 32.4 mm
- net RST: track 136.3 -> 138.7 mm
- net MOSI: track 48.4 -> 50.2 mm
- net SCK: track 36.6 -> 38.3 mm
Changed lines of the file:
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@@
 <?xml version="1.0" encoding="utf-8"?>
 <!DOCTYPE eagle SYSTEM "eagle.dtd">
-<eagle version="7.4.0">
+<eagle version="7.5.0">
 <drawing>
 <settings>
@@
 <layers>
 <layer number="1" name="Top" color="4" fill="1" visible="yes" active="yes"/>
-<layer number="16" name="Bottom" color="1" fill="1" visible="no" active="yes"/>
+<layer number="16" name="Bottom" color="1" fill="1" visible="yes" active="yes"/>
 <layer number="17" name="Pads" color="2" fill="1" visible="yes" active="yes"/>
 <layer number="18" name="Vias" color="2" fill="1" visible="yes" active="yes"/>
@@
 <attribute name="VARIANT" value="" x="44.5" y="36.5" size="1.778" layer="27" rot="R90" display="off"/>
 </element>
-<element name="JP2" library="fab" package="2X03SMD" value="" x="-4.25" y="5.6"/>
+<element name="JP1" library="pinhead" package="2X03" value="" x="43.4" y="26.6" rot="MR270"/>
 </elements>
 <signals>
@@
 <contactref element="C3" pad="2"/>
 <contactref element="D2" pad="8"/>
+<contactref element="JP1" pad="2"/>
 <wire x1="44.1198" y1="42.7482" x2="44.1" y2="43.378" width="0.254" layer="1"/>
 <wire x1="42.0092" y1="29.2608" x2="39.3" y2="29.2608" width="0.254" layer="1"/>
@@
 <wire x1="60.5" y1="33.9118" x2="59.436" y2="34.9758" width="0.254" layer="1" curve="90"/>
 <wire x1="40.5194" y1="26.1306" x2="40.5194" y2="27.7806" width="0.254" layer="1"/>
+<wire x1="42.0092" y1="29.2608" x2="42.13" y2="29.14" width="0.254" layer="1"/>
 <wire x1="40.5" y1="27.8" x2="40.5" y2="28.0608" width="0.254" layer="1"/>
 <wire x1="40.5" y1="28.0608" x2="39.3" y2="29.2608" width="0.254" layer="1" curve="90"/>
@@
 <wire x1="40.5194" y1="27.7806" x2="40.5" y2="27.8" width="0.254" layer="1" curve="90"/>
 <wire x1="40.5194" y1="26.1306" x2="41.3" y2="25.35" width="0.254" layer="1" curve="90"/>
-<contactref element="JP2" pad="2"/>
-<wire x1="-1.3925" y1="8.14" x2="35.7" y2="30.1798" width="0" layer="19" extent="1-1"/>
 </signal>
 <signal name="RST">
 <contactref element="R1" pad="1"/>
+<contactref element="JP1" pad="5"/>
 <contactref element="S1" pad="3"/>
 <contactref element="IC1" pad="29"/>
@@
 <wire x1="73.8" y1="40.7" x2="73.8" y2="50.4" width="0.254" layer="1"/>
 <wire x1="73.8" y1="50.4" x2="71.8" y2="52.9" width="0.254" layer="1" curve="90"/>
+<wire x1="44.67" y1="24.06" x2="44.67" y2="21.63" width="0.254" layer="1"/>
 <wire x1="44.67" y1="21.63" x2="47.2" y2="19.6" width="0.254" layer="1" curve="90"/>
 <wire x1="47.2" y1="19.6" x2="65.3" y2="19.6" width="0.254" layer="1"/>
@@
 <wire x1="52.4" y1="52.9" x2="71.8" y2="52.9" width="0.254" layer="1"/>
 <wire x1="49.8" y1="50.3" x2="52.4" y2="52.9" width="0.254" layer="1" curve="-90"/>
-<contactref element="JP2" pad="5"/>
-<wire x1="-7.1075" y1="3.06" x2="44.67" y2="21.63" width="0" layer="19" extent="1-1"/>
 </signal>
 <signal name="N$3">
@@
 <contactref element="IC1" pad="15"/>
 <contactref element="D2" pad="4"/>
+<contactref element="JP1" pad="4"/>
 <wire x1="60.7456" y1="21.6456" x2="49.0544" y2="21.6456" width="0.254" layer="1"/>
 <wire x1="61.5434" y1="25.6066" x2="61.5434" y2="23.0886" width="0.254" layer="1"/>
@@
 <wire x1="47.9" y1="26.9" x2="46.95" y2="27.85" width="0.254" layer="1" curve="90"/>
 <wire x1="46.95" y1="27.85" x2="43.38" y2="27.85" width="0.254" layer="1"/>
+<wire x1="43.38" y1="27.85" x2="42.13" y2="26.6" width="0.254" layer="1" curve="90"/>
 <wire x1="61.5434" y1="25.6066" x2="60.75" y2="26.4" width="0.254" layer="1" curve="90"/>
 <wire x1="60.75" y1="26.4" x2="59.35" y2="27" width="0.254" layer="1" curve="-48.455236"/>
 <wire x1="59.35" y1="27" x2="57.8" y2="29.1" width="0.254" layer="1" curve="-35.069943"/>
-<contactref element="JP2" pad="4"/>
-<wire x1="-1.3925" y1="5.6" x2="43.38" y2="27.85" width="0" layer="19" extent="1-1"/>
 </signal>
 <signal name="MISO">
 <contactref element="IC1" pad="16"/>
 <contactref element="D2" pad="5"/>
+<contactref element="JP1" pad="1"/>
 <wire x1="56.2356" y1="32.4612" x2="56.2" y2="32.5804" width="0.254" layer="1"/>
 <wire x1="58.9028" y1="22.3028" x2="49.6062" y2="22.3028" width="0.254" layer="1"/>
+<wire x1="44.67" y1="29.14" x2="47.36" y2="29.14" width="0.254" layer="1"/>
 <wire x1="47.36" y1="29.14" x2="48.7" y2="27.8" width="0.254" layer="1" curve="-90"/>
 <wire x1="48.7" y1="27.8" x2="48.7" y2="23.209" width="0.254" layer="1"/>
@@
 <wire x1="60.27" y1="24.63" x2="60.27" y2="24.4" width="0.254" layer="1"/>
 <wire x1="60.27" y1="24.63" x2="56.2" y2="28.7" width="0.254" layer="1"/>
-<contactref element="JP2" pad="1"/>
-<wire x1="-7.1075" y1="8.14" x2="48.7" y2="23.209" width="0" layer="19" extent="1-1"/>
 </signal>
 <signal name="SCK">
@@
 <contactref element="IC1" pad="17"/>
 <contactref element="D2" pad="6"/>
+<contactref element="JP1" pad="3"/>
 <wire x1="60.8076" y1="28.3464" x2="61" y2="28.178" width="0.254" layer="1"/>
 <wire x1="61.8884" y1="20.9884" x2="48.5116" y2="20.9884" width="0.254" layer="1"/>
 <wire x1="61.0362" y1="28.1178" x2="61" y2="28.178" width="0.254" layer="1"/>
 <wire x1="62.6364" y1="24.4602" x2="62.81" y2="24.4" width="0.254" layer="1"/>
+<wire x1="44.67" y1="26.6" x2="46.4" y2="26.6" width="0.254" layer="1"/>
 <wire x1="59.2" y1="29.2" x2="59.2" y2="33.6" width="0.254" layer="1"/>
 <wire x1="46.4" y1="26.6" x2="47.1" y2="25.9" width="0.254" layer="1" curve="-90"/>
@@
 <wire x1="61.0362" y1="28.1178" x2="62.81" y2="26.344" width="0.254" layer="1"/>
 <wire x1="62.81" y1="26.344" x2="62.81" y2="24.4" width="0.254" layer="1"/>
-<contactref element="JP2" pad="3"/>
-<wire x1="-7.1075" y1="5.6" x2="47.1" y2="22.4" width="0" layer="19" extent="1-1"/>
 </signal>
 <signal name="N$23">
@@
 <wire x1="50.8" y1="43.3" x2="48.7" y2="45.4" width="0.254" layer="1" curve="-90"/>
 <wire x1="48.7" y1="45.4" x2="48.7" y2="48.6" width="0.254" layer="1"/>
+</signal>
+<signal name="N$1">
+<contactref element="IC1" pad="8"/>
+<contactref element="U$2" pad="1"/>
+<wire x1="45.9486" y1="34.29" x2="48.9204" y2="34.29" width="0.254" layer="1"/>
+<wire x1="48.9204" y1="34.29" x2="48.9804" y2="34.2" width="0.254" layer="1"/>
+<wire x1="45.0342" y1="35.2044" x2="44.5" y2="35.15" width="0.254" layer="1"/>
+<wire x1="45.0342" y1="35.2044" x2="45.9486" y2="34.29" width="0.254" layer="1" curve="90"/>
+</signal>
+<signal name="N$9">
+<contactref element="IC1" pad="7"/>
+<contactref element="U$2" pad="3"/>
+<wire x1="48.1242" y1="34.9758" x2="49.149" y2="34.9758" width="0.254" layer="1"/>
+<wire x1="49.149" y1="34.9758" x2="49.2344" y2="35" width="0.254" layer="1"/>
+<wire x1="48.1242" y1="34.9758" x2="48.1" y2="35" width="0.254" layer="1"/>
+<wire x1="48.1" y1="35" x2="48" y2="35" width="0.254" layer="1"/>
+<wire x1="44.5" y1="37.85" x2="46.75" y2="37.85" width="0.254" layer="1"/>
+<wire x1="46.75" y1="37.85" x2="47.2" y2="37.2" width="0.254" layer="1" curve="-68.760689"/>
+<wire x1="47.2" y1="37.2" x2="47.2" y2="35.6" width="0.254" layer="1"/>
+<wire x1="47.2" y1="35.6" x2="48" y2="35" width="0.254" layer="1" curve="90"/>
 </signal>
 <signal name="N$10">
@@
 <contactref element="U$2" pad="2"/>
 <contactref element="D2" pad="7"/>
+<contactref element="JP1" pad="6"/>
 <polygon width="0.4064" layer="16">
 <vertex x="36.8" y="51.8"/>
@@
 <wire x1="47.7" y1="38.2" x2="49.2344" y2="38.2" width="0.254" layer="1"/>
 <wire x1="41.8" y1="36.8" x2="41.3" y2="37.3" width="0.254" layer="1" curve="-90"/>
-<contactref element="JP2" pad="6"/>
-<wire x1="65.35" y1="24.4" x2="64.4" y2="31.022" width="0" layer="19" extent="1-1"/>
-<wire x1="57.5656" y1="37.4" x2="64.3" y2="35" width="0" layer="19" extent="1-1"/>
-<wire x1="46.7" y1="46.222" x2="46.9" y2="39" width="0" layer="19" extent="1-1"/>
-<wire x1="39.1" y1="24" x2="42.1" y2="36.5" width="0" layer="19" extent="1-1"/>
-<wire x1="-1.3925" y1="3.06" x2="39.1" y2="24" width="0" layer="19" extent="1-1"/>
-</signal>
-<signal name="N$16">
-<contactref element="IC1" pad="8"/>
-<contactref element="U$2" pad="3"/>
-<wire x1="44.5" y1="37.85" x2="48.9804" y2="34.2" width="0" layer="19" extent="1-1"/>
-</signal>
-<signal name="N$1">
-<contactref element="IC1" pad="7"/>
-<contactref element="U$2" pad="1"/>
-<wire x1="44.5" y1="35.15" x2="49.2344" y2="35" width="0" layer="19" extent="1-1"/>
+</signal>
+<signal name="S$1">
+<wire x1="42.05" y1="24.05" x2="39.15" y2="24.05" width="0.4064" layer="1"/>
+<wire x1="39.15" y1="24.05" x2="39.15" y2="24" width="0.4064" layer="1"/>
 </signal>
 </signals>
